Commit message: repair gazebo simulation

File: movensys_navigation_description/urdf/diffbot/control.xacro (robot description, xacro)
@@ -25,5 +25,5 @@
 		</joint>
 		<joint name="drivewheel_right_joint">
-    		<command_interface name="position"/>
+    		<command_interface name="velocity"/>
     		<state_interface name="velocity"/>
     	</joint>

File: movensys_navigation_description/urdf/diffbot/diffbot.xacro (robot description, xacro)
@@ -5,5 +5,5 @@
 		<visual>
 			<geometry>
-				<box size="0.64 0.52 0.1"></box>
+				<box size="0.7 0.6 0.1"></box>
 			</geometry>
 			<origin rpy="0 0 0" xyz="0 0 0"></origin>
@@ -14,5 +14,5 @@
 		<collision>
 			<geometry>
-				<box size="0.64 0.52 0.1"></box>
+				<box size="0.7 0.6 0.1"></box>
 			</geometry>
 			<origin rpy="0 0 0" xyz="0 0 0"></origin>
