Commit message: add gazebo perception

File: movensys_navigation_description/urdf/diffbot/diffbot.xacro (robot description, xacro)
@@ -2,5 +2,5 @@
 <robot xmlns:xacro="http://www.ros.org/wiki/xacro">
 <xacro:macro name="diffbot">
-  <link name="base_link">
+  	<link name="base_link">
 		<visual>
 			<geometry>
@@ -8,7 +8,7 @@
 			</geometry>
 			<origin rpy="0 0 0" xyz="0 0 0"></origin>
-      <material name="">
-        <color rgba="1 1 1 1" />
-      </material>
+      		<material name="">
+        		<color rgba="1 1 1 1" />
+      		</material>
 		</visual>
 		<collision>
@@ -38,5 +38,5 @@
 			<origin rpy="0 0 0" xyz="0 0 0"></origin>
 		</visual>
-    <collision>
+    	<collision>
 			<geometry>
 				<sphere radius="0.06"></sphere>
@@ -64,5 +64,5 @@
 			<origin rpy="0 0 0" xyz="0 0 0"></origin>
 		</visual>
-    <collision>
+    	<collision>
 			<geometry>
 				<sphere radius="0.06"></sphere>

File: movensys_navigation_description/urdf/diffbot/movensys_navigation.gazebo.xacro (robot description, xacro)
@@ -4,4 +4,6 @@
     <xacro:include filename="$(find movensys_navigation_description)/urdf/diffbot/control.xacro" />
     <xacro:include filename="$(find movensys_navigation_description)/urdf/diffbot/transmission.xacro" />
+    <xacro:include filename="$(find movensys_navigation_description)/urdf/diffbot/perception.xacro" />
+    <xacro:include filename="$(find movensys_navigation_description)/urdf/diffbot/perception.gazebo" />
     <link name="base_footprint"/>
     <joint name="base_link_joint" type="fixed">

Commit message: add isaacsim

File: movensys_navigation_description/urdf/diffbot/diffbot.xacro (robot description, xacro)
@@ -25,5 +25,5 @@
 		</inertial>
 	</link>
-	<joint name="castor_rear_right_joint" type="continuous">
+	<joint name="castor_rear_right_joint" type="fixed">
 		<parent link="base_link"></parent>
 		<child link="castor_rear_right"></child>
@@ -51,5 +51,5 @@
 		</inertial>
 	</link>
-	<joint name="castor_rear_left_joint" type="continuous">
+	<joint name="castor_rear_left_joint" type="fixed">
 		<parent link="base_link"></parent>
 		<child link="castor_rear_left"></child>
