Commit message: add rsp arg

File: movensys_navigation_description/urdf/diffbot/movensys_navigation.gazebo.xacro (robot description, xacro)
@@ -1,8 +1,7 @@
 <?xml version="1.0"?>
 <robot name="movensys_navigation" xmlns:xacro="http://www.ros.org/wiki/xacro">
-    <xacro:include filename="$(find movensys_navigation_description)/urdf/diffbot/diffbot.xacro" />
+    <xacro:include filename="$(find movensys_navigation_description)/urdf/diffbot/movensys_navigation.xacro" />
     <xacro:include filename="$(find movensys_navigation_description)/urdf/diffbot/control.xacro" />
     <xacro:include filename="$(find movensys_navigation_description)/urdf/diffbot/transmission.xacro" />
-    <xacro:include filename="$(find movensys_navigation_description)/urdf/diffbot/perception.xacro" />
     <xacro:include filename="$(find movensys_navigation_description)/urdf/diffbot/perception.gazebo" />
     <link name="base_footprint"/>

File: movensys_navigation_description/urdf/diffbot/movensys_navigation.urdf (robot description, URDF)
Before this commit: robot movensys_navigation, 6 links, 5 joints
Links:
- added link imu_link, mass 0.001; visual box size=0.001 0.001 0.001
- added link lidar_front_left_link, mass 0.130; collision cylinder length=0.1 radius=0.05; visual cylinder length=0.1 radius=0.05
- added link lidar_rear_right_link, mass 0.130; collision cylinder length=0.1 radius=0.05; visual cylinder length=0.1 radius=0.05
- added link ray_front_left_link; visual box size=0.001 0.001 0.001
- added link ray_rear_right_link; visual box size=0.001 0.001 0.001
- added link value_link; visual box size=0.001 0.001 0.001
Joints:
- added joint imu_joint: type fixed, parent base_link, child imu_link, origin xyz=0 0 0 rpy=0 0 0
- added joint imu_to_value: type fixed, parent imu_link, child value_link, origin xyz=0 0 0 rpy=0 0 0
- added joint lidar_front_left_joint: type fixed, parent base_link, child lidar_front_left_link, origin xyz=0.3 0.25 0.185 rpy=0 0 0.7853981633974484, axis 0 0 1
- added joint lidar_rear_right_joint: type fixed, parent base_link, child lidar_rear_right_link, origin xyz=-0.3 -0.25 0.185 rpy=0 0 -2.356194490192345, axis 0 0 1
- added joint ray_front_left_joint: type fixed, parent lidar_front_left_link, child ray_front_left_link, origin xyz=0 0 0 rpy=0 0 0
- added joint ray_rear_right_joint: type fixed, parent lidar_rear_right_link, child ray_rear_right_link, origin xyz=0 0 0 rpy=0 0 0

File: movensys_navigation_description/urdf/diffbot/movensys_navigation.xacro (robot description, xacro)
@@ -2,4 +2,5 @@
 <robot name="movensys_navigation" xmlns:xacro="http://www.ros.org/wiki/xacro">
     <xacro:include filename="$(find movensys_navigation_description)/urdf/diffbot/diffbot.xacro" />
+    <xacro:include filename="$(find movensys_navigation_description)/urdf/diffbot/perception.xacro" />
     <link name="base_footprint"/>
     <joint name="base_link_joint" type="fixed">

Commit message: repair twist stamped

File: movensys_navigation_description/urdf/diffbot/movensys_navigation.gazebo.xacro (robot description, xacro)
@@ -5,10 +5,3 @@
     <xacro:include filename="$(find movensys_navigation_description)/urdf/diffbot/transmission.xacro" />
     <xacro:include filename="$(find movensys_navigation_description)/urdf/diffbot/perception.gazebo" />
-    <link name="base_footprint"/>
-    <joint name="base_link_joint" type="fixed">
-        <origin xyz="0 0 0.095" rpy="0 0 0" />
-        <parent link="base_footprint" />
-        <child link="base_link" />
-    </joint>
-    <xacro:diffbot />
 </robot>
