Commit message: manual diffbot sim and hil good

File: movensys_navigation_description/urdf/diffbot/movensys_navigation.urdf (robot description, URDF)
Before this commit: robot movensys_navigation, 12 links, 11 joints
Links:
- removed link base_footprint
Joints:
- removed joint base_link_joint

File: movensys_navigation_description/urdf/diffbot/movensys_navigation.xacro (robot description, xacro)
@@ -3,10 +3,4 @@
     <xacro:include filename="$(find movensys_navigation_description)/urdf/diffbot/diffbot.xacro" />
     <xacro:include filename="$(find movensys_navigation_description)/urdf/diffbot/perception.xacro" />
-    <link name="base_footprint"/>
-    <joint name="base_link_joint" type="fixed">
-        <origin xyz="0 0 0.095" rpy="0 0 0" />
-        <parent link="base_footprint" />
-        <child link="base_link" />
-    </joint>
     <xacro:diffbot />
 </robot>
