Commit message: repair transform issue

File: movensys_navigation_description/urdf/diffbot/movensys_navigation.urdf (robot description, URDF)
Before this commit: robot movensys_navigation, 11 links, 10 joints
Links:
- added link camera_front_link, mass 0.072; collision box size=0.025 0.09 0.025; visual box size=0.025 0.09 0.025
Joints:
- added joint camera_joint: type fixed, parent base_link, child camera_front_link, origin xyz=0.4 0.0 0.17 rpy=0 0 0

Commit message: repair camera tf transform

File: movensys_navigation_description/urdf/diffbot/movensys_navigation.urdf (robot description, URDF)
Before this commit: robot movensys_navigation, 12 links, 11 joints
Links:
- added link camera_front_infra1_optical_frame
- added link camera_front_infra2_optical_frame
Joints:
- added joint camera_front_infra1_optical_joint: type fixed, parent camera_front_link, child camera_front_infra1_optical_frame, origin xyz=0 0 0 rpy=-1.5707963 0 -1.5707963
- added joint camera_front_infra2_optical_joint: type fixed, parent camera_front_link, child camera_front_infra2_optical_frame, origin xyz=0 -0.095 0 rpy=-1.5707963 0 -1.5707963

File: movensys_navigation_description/urdf/diffbot/perception.xacro (robot description, xacro)
@@ -137,3 +137,18 @@
         </collision>
     </link>
+    <xacro:arg name="urdf_camera_optical_tf" default="true"/>
+    <xacro:if value="$(arg urdf_camera_optical_tf)">
+        <joint name="camera_front_infra1_optical_joint" type="fixed">
+            <parent link="camera_front_link"/>
+            <child link="camera_front_infra1_optical_frame"/>
+            <origin xyz="0 0 0" rpy="-1.5707963 0 -1.5707963"/>
+        </joint>
+        <link name="camera_front_infra1_optical_frame"/>
+        <joint name="camera_front_infra2_optical_joint" type="fixed">
+            <parent link="camera_front_link"/>
+            <child link="camera_front_infra2_optical_frame"/>
+            <origin xyz="0 -0.095 0" rpy="-1.5707963 0 -1.5707963"/>
+        </joint>
+        <link name="camera_front_infra2_optical_frame"/>
+    </xacro:if>
 </robot>
