Commit message: add cuvslam

File: movensys_navigation_description/urdf/diffbot/perception.xacro (robot description, xacro)
@@ -110,3 +110,30 @@
         </visual>
     </link>
+    <joint name="camera_joint" type="fixed">
+        <parent link="base_link"/>
+        <child link="camera_front_link"/>
+        <origin rpy="0 0 0" xyz="0.4 0.0 0.17"/>
+    </joint>
+    <link name="camera_link">
+        <inertial>
+            <mass value="0.072"/>
+            <origin rpy="0 0 0" xyz="0 0 0"/>
+            <inertia ixx="0.0001" ixy="0" ixz="0" iyy="0.0001" iyz="0" izz="0.0001"/>
+        </inertial>
+        <visual>
+            <origin rpy="0 0 0" xyz="0 0 0"/>
+            <geometry>
+                <box size="0.025 0.09 0.025"/>
+            </geometry>
+            <material name="">
+                <color rgba="0.1 0.1 0.1 1"/>
+            </material>
+        </visual>
+        <collision>
+            <origin rpy="0 0 0" xyz="0 0 0"/>
+            <geometry>
+                <box size="0.025 0.09 0.025"/>
+            </geometry>
+        </collision>
+    </link>
 </robot>

Commit message: repair cuVslam

File: movensys_navigation_description/urdf/diffbot/perception.xacro (robot description, xacro)
@@ -115,5 +115,5 @@
         <origin rpy="0 0 0" xyz="0.4 0.0 0.17"/>
     </joint>
-    <link name="camera_link">
+    <link name="camera_front_link">
         <inertial>
             <mass value="0.072"/>
